Commit message: second commite

File: src/xingtian_dynamics/urdf/xingtian_urdf.xacro (robot description, xacro)
@@ -30,7 +30,7 @@
       <kp>1000000.0</kp>
       <kd>1.0</kd>
-      <minDepth>0.00</minDepth>
-      <maxVel>2.0</maxVel>
-      <fdir1>1 0 0 </fdir1>     <!-- force direaction  -->
+      <!-- <minDepth>0.00</minDepth>
+      <maxVel>2.0</maxVel> -->
+      <!-- <fdir1>1 0 0 </fdir1>     force direaction  -->
  </gazebo>
  <gazebo reference = "zht_qubing">
@@ -39,7 +39,7 @@
       <kp>1000000.0</kp>
       <kd>1.0</kd>
-      <minDepth>0.00</minDepth>
-      <maxVel>2.0</maxVel>
-      <fdir1>1 0 0 </fdir1>     <!-- force direaction  -->
+      <!-- <minDepth>0.00</minDepth>
+      <maxVel>2.0</maxVel> -->
+      <!-- <fdir1>1 0 0 </fdir1>     force direaction  -->
  </gazebo>
  <gazebo reference = "zht_dianjizhou">
@@ -48,16 +48,17 @@
       <kp>1000000.0</kp>
       <kd>1.0</kd>
-      <minDepth>0.00</minDepth>
-      <maxVel>2.0</maxVel>
-      <fdir1>1 0 0 </fdir1>     <!-- force direaction  -->
+      <!-- <minDepth>0.00</minDepth>
+      <maxVel>2.0</maxVel> -->
+      <!-- <fdir1>1 0 0 </fdir1>     force direaction  -->
  </gazebo>
  <gazebo reference = "zht_wheel">
-      <mu1>0.8</mu1>
+      <mu1>0.6</mu1>
       <mu2>0.6</mu2>
       <kp>1000000.0</kp>
       <kd>1.0</kd>
-      <minDepth>0.00</minDepth>
-      <maxVel>2.0</maxVel>
-      <fdir1>1 0 0 </fdir1>     <!-- force direaction  -->
+      <self_collide>1</self_collide>
+      <!-- <minDepth>0.00</minDepth>
+      <maxVel>2.0</maxVel> -->
+      <!-- <fdir1>1 0 0 </fdir1>     force direaction  -->
  </gazebo>
  <gazebo reference = "yht_yao">  <!--从上往下-->
@@ -66,7 +67,7 @@
       <kp>1000000.0</kp>
       <kd>1.0</kd>
-      <minDepth>0.00</minDepth>
-      <maxVel>2.0</maxVel>
-      <fdir1>1 0 0 </fdir1>     <!-- force direaction  -->
+      <!-- <minDepth>0.00</minDepth>
+      <maxVel>2.0</maxVel> -->
+      <!-- <fdir1>1 0 0 </fdir1>     force direaction  -->
  </gazebo>
  <gazebo reference = "yht_qubing">
@@ -75,7 +76,7 @@
       <kp>1000000.0</kp>
       <kd>1.0</kd>
-      <minDepth>0.00</minDepth>
-      <maxVel>2.0</maxVel>
-      <fdir1>1 0 0 </fdir1>     <!-- force direaction  -->
+      <!-- <minDepth>0.00</minDepth>
+      <maxVel>2.0</maxVel> -->
+      <!-- <fdir1>1 0 0 </fdir1>     force direaction  -->
  </gazebo>
  <gazebo reference = "yht_dianjizhou">
@@ -84,16 +85,17 @@
       <kp>1000000.0</kp>
       <kd>1.0</kd>
-      <minDepth>0.00</minDepth>
-      <maxVel>2.0</maxVel>
-      <fdir1>1 0 0 </fdir1>     <!-- force direaction  -->
+      <!-- <minDepth>0.00</minDepth>
+      <maxVel>2.0</maxVel> -->
+      <!-- <fdir1>1 0 0 </fdir1>     force direaction  -->
  </gazebo>
  <gazebo reference = "yht_wheel">
-      <mu1>0.8</mu1>
+      <mu1>0.6</mu1>
       <mu2>0.6</mu2>
       <kp>1000000.0</kp>
       <kd>1.0</kd>
-      <minDepth>0.00</minDepth>
-      <maxVel>2.0</maxVel>
-      <fdir1>1 0 0 </fdir1>     <!-- force direaction  -->
+      <self_collide>1</self_collide>
+      <!-- <minDepth>0.00</minDepth>
+      <maxVel>2.0</maxVel> -->
+      <!-- <fdir1>1 0 0 </fdir1>     force direaction  -->
  </gazebo>
  <gazebo reference = "yqt_yao">  <!--从上往下-->
@@ -102,7 +104,7 @@
       <kp>1000000.0</kp>
       <kd>1.0</kd>
-      <minDepth>0.00</minDepth>
-      <maxVel>2.0</maxVel>
-      <fdir1>1 0 0 </fdir1>     <!-- force direaction  -->
+      <!-- <minDepth>0.00</minDepth>
+      <maxVel>2.0</maxVel> -->
+      <!-- <fdir1>1 0 0 </fdir1>     force direaction  -->
  </gazebo>
  <gazebo reference = "yqt_qubing">
@@ -111,7 +113,7 @@
       <kp>1000000.0</kp>
       <kd>1.0</kd>
-      <minDepth>0.00</minDepth>
-      <maxVel>2.0</maxVel>
-      <fdir1>1 0 0 </fdir1>     <!-- force direaction  -->
+      <!-- <minDepth>0.00</minDepth>
+      <maxVel>2.0</maxVel> -->
+      <!-- <fdir1>1 0 0 </fdir1>     force direaction  -->
  </gazebo>
  <gazebo reference = "yqt_dianjizhou">
@@ -120,16 +122,17 @@
       <kp>1000000.0</kp>
       <kd>1.0</kd>
-      <minDepth>0.00</minDepth>
-      <maxVel>2.0</maxVel>
-      <fdir1>1 0 0 </fdir1>     <!-- force direaction  -->
+      <!-- <minDepth>0.00</minDepth>
+      <maxVel>2.0</maxVel> -->
+      <!-- <fdir1>1 0 0 </fdir1>     force direaction  -->
  </gazebo>
  <gazebo reference = "yqt_wheel">
-      <mu1>0.8</mu1>
+      <mu1>0.6</mu1>
       <mu2>0.6</mu2>
       <kp>1000000.0</kp>
       <kd>1.0</kd>
-      <minDepth>0.00</minDepth>
-      <maxVel>2.0</maxVel>
-      <fdir1>1 0 0 </fdir1>     <!-- force direaction  -->
+      <self_collide>1</self_collide>
+      <!-- <minDepth>0.00</minDepth>
+      <maxVel>2.0</maxVel> -->
+      <!-- <fdir1>1 0 0 </fdir1>     force direaction  -->
  </gazebo>
  <gazebo reference = "zqt_yao">  <!--从上往下-->
@@ -138,7 +141,7 @@
       <kp>1000000.0</kp>
       <kd>1.0</kd>
-      <minDepth>0.00</minDepth>
-      <maxVel>2.0</maxVel>
-      <fdir1>1 0 0 </fdir1>     <!-- force direaction  -->
+      <!-- <minDepth>0.00</minDepth>
+      <maxVel>2.0</maxVel> -->
+      <!-- <fdir1>1 0 0 </fdir1>     force direaction  -->
  </gazebo>
   <gazebo reference = "zqt_qubing">
@@ -147,7 +150,7 @@
       <kp>1000000.0</kp>
       <kd>1.0</kd>
-      <minDepth>0.00</minDepth>
-      <maxVel>2.0</maxVel>
-      <fdir1>1 0 0 </fdir1>     <!-- force direaction  -->
+      <!-- <minDepth>0.00</minDepth>
+      <maxVel>2.0</maxVel> -->
+      <!-- <fdir1>1 0 0 </fdir1>     force direaction  -->
   </gazebo>
   <gazebo reference = "zqt_dianjizhou">
@@ -156,16 +159,17 @@
       <kp>1000000.0</kp>
       <kd>1.0</kd>
-      <minDepth>0.00</minDepth>
-      <maxVel>2.0</maxVel>
-      <fdir1>1 0 0 </fdir1>     <!-- force direaction  -->
+      <!-- <minDepth>0.00</minDepth>
+      <maxVel>2.0</maxVel> -->
+      <!-- <fdir1>1 0 0 </fdir1>     force direaction  -->
   </gazebo>
   <gazebo reference = "zqt_wheel">
-      <mu1>0.8</mu1>
+      <mu1>0.6</mu1>
       <mu2>0.6</mu2>
       <kp>1000000.0</kp>
       <kd>1.0</kd>
-      <minDepth>0.00</minDepth>
-      <maxVel>2.0</maxVel>
-      <fdir1>1 0 0 </fdir1>     <!-- force direaction  -->
+      <self_collide>1</self_collide>
+      <!-- <minDepth>0.00</minDepth>
+      <maxVel>2.0</maxVel> -->
+      <!-- <fdir1>1 0 0 </fdir1>     force direaction  -->
   </gazebo>
   <!-- sensor -->
@@ -403,28 +407,4 @@
       <provideFeedback>true</provideFeedback>
   </gazebo>
-<!-- 虚拟传感器 -->
-   <!-- <gazebo  reference="fake_LF_joint1">
-      <provideFeedback>true</provideFeedback>
-  </gazebo>
-   <gazebo  reference="fake_LR_joint1">
-      <provideFeedback>true</provideFeedback>
-  </gazebo>
-   <gazebo  reference="fake_RR_joint1">
-      <provideFeedback>true</provideFeedback>
-  </gazebo>
-   <gazebo  reference="fake_RF_joint1">
-      <provideFeedback>true</provideFeedback>
-  </gazebo> -->
-  <!-- <gazebo>
-        <plugin filename="/opt/ros/noetic/lib/libgazebo_ros_ft_sensor.so" name="ft_sensor">
-            <updateRate>300</updateRate>
-            <topicName>xingtian/force_LR_wheel</topicName>
-            <jointName>zht_joint1</jointName>
-            <force_torque>
-              <frame>world</frame>
-              <measure_direction>child_to_parent</measure_direction>
-            </force_torque>
-        </plugin>
-  </gazebo>  -->
   <gazebo>
         <plugin filename="/opt/ros/noetic/lib/libgazebo_ros_ft_sensor.so" name="ft_sensor">
@@ -819,44 +799,5 @@
       </actuator>
     </transmission>
-     <!-- <transmission name = "trans4">
-      <type>transmission_interface/SimpleTransmission</type>
-      <joint name = "zqt_joint4">
-        <hardwareInterface>hardware_interface/PositonJointInterface</hardwareInterface>
-      </joint>
-      <actuator name = "effort_motor">
-        <hardwareInterface>hardware_interface/PositonJointInterface</hardwareInterface>
-        <mechanicalReduction>1</mechanicalReduction>
-      </actuator>
-    </transmission>
-    <transmission name = "trans4">
-      <type>transmission_interface/SimpleTransmission</type>
-      <joint name = "zht_joint4">
-        <hardwareInterface>hardware_interface/PositonJointInterface</hardwareInterface>
-      </joint>
-      <actuator name = "position_motor">
-        <hardwareInterface>hardware_interface/PositonJointInterface</hardwareInterface>
-        <mechanicalReduction>1</mechanicalReduction>
-      </actuator>
-    </transmission>
-    <transmission name = "trans4">
-      <type>transmission_interface/SimpleTransmission</type>
-      <joint name = "yht_joint4">
-        <hardwareInterface>hardware_interface/PositionJointInterface</hardwareInterface>
-      </joint>
-      <actuator name = "position_motor">
-        <hardwareInterface>hardware_interface/PositonJointInterface</hardwareInterface>
-        <mechanicalReduction>1</mechanicalReduction>
-      </actuator>
-    </transmission>
-    <transmission name = "trans4">
-      <type>transmission_interface/SimpleTransmission</type>
-      <joint name = "yqt_joint4">
-        <hardwareInterface>hardware_interface/PositionJointInterface</hardwareInterface>
-      </joint>
-      <actuator name = "position_motor">
-        <hardwareInterface>hardware_interface/PositionJointInterface</hardwareInterface>
-        <mechanicalReduction>1</mechanicalReduction>
-      </actuator>
-    </transmission> -->
+<!--
   <xacro:macro name = "joint_setup_block" params = "joint_name">
     <gazebo reference = "${joint_name}">
@@ -879,5 +820,5 @@
   <xacro:joint_setup_block joint_name = "yqt_joint2"/>
   <xacro:joint_setup_block joint_name = "yqt_joint3"/>
-  <xacro:joint_setup_block joint_name = "yqt_joint4"/>
+  <xacro:joint_setup_block joint_name = "yqt_joint4"/> -->
   <!--link and joint-->
   <link
@@ -1067,5 +1008,5 @@
       </material>
     </visual>
-    <collision>
+    <!-- <collision>
       <origin
         xyz="0 0 0"
@@ -1075,5 +1016,5 @@
           filename="package://xingtian/meshes/meshes_s/zht_yao.STL" />
       </geometry>
-    </collision>
+    </collision> -->
   </link>
   <joint
@@ -1128,5 +1069,5 @@
       </material>
     </visual>
-    <collision>
+    <!-- <collision>
       <origin
         xyz="0 0 0"
@@ -1136,5 +1077,5 @@
           filename="package://xingtian/meshes/meshes_s/zht_qubing.STL" />
       </geometry>
-    </collision>
+    </collision> -->
   </link>
   <joint
@@ -1153,5 +1094,5 @@
       <update_rate>300</update_rate>
     </sensor>
-    <dynamics damping="0.1" friction="0.1"/>
+    <!-- <dynamics damping="0.1" friction="0.1"/> -->
     <limit
       lower="-3.14"
@@ -1190,5 +1131,5 @@
       </material>
     </visual>
-    <collision>
+    <!-- <collision>
       <origin
         xyz="0 0 0"
@@ -1198,5 +1139,5 @@
           filename="package://xingtian/meshes/meshes_s/zht_dianjizhou.STL" />
       </geometry>
-    </collision>
+    </collision> -->
   </link>
   <joint
@@ -1212,5 +1153,5 @@
     <axis
       xyz="0 -1 0" />
-    <dynamics damping="0.1" friction="0.1"/>
+    <!-- <dynamics damping="0.1" friction="0.1"/> -->
     <limit
       lower="-3.14"
@@ -1305,5 +1246,5 @@
       </material>
     </visual>
-    <collision>
+    <!-- <collision>
       <origin
         xyz="0 0 0"
@@ -1313,5 +1254,5 @@
           filename="package://xingtian/meshes/meshes_s/yht_yao.STL" />
       </geometry>
-    </collision>
+    </collision> -->
   </link>
   <joint
@@ -1366,5 +1307,5 @@
       </material>
     </visual>
-    <collision>
+    <!-- <collision>
       <origin
         xyz="0 0 0"
@@ -1374,5 +1315,5 @@
           filename="package://xingtian/meshes/meshes_s/yht_qubing.STL" />
       </geometry>
-    </collision>
+    </collision> -->
   </link>
   <joint
@@ -1391,5 +1332,5 @@
       <update_rate>300</update_rate>
     </sensor>
-    <dynamics damping="0.1" friction="0.1"/>
+    <!-- <dynamics damping="0.1" friction="0.1"/> -->
     <limit
       lower="-3.14"
@@ -1429,5 +1370,5 @@
       </material>
     </visual>
-    <collision>
+    <!-- <collision>
       <origin
         xyz="0 0 0"
@@ -1437,5 +1378,5 @@
           filename="package://xingtian/meshes/meshes_s/yht_dianjizhou.STL" />
       </geometry>
-    </collision>
+    </collision> -->
   </link>
   <joint
@@ -1455,5 +1396,5 @@
       <update_rate>300</update_rate>
     </sensor>
-    <dynamics damping="0.1" friction="0.1"/>
+    <!-- <dynamics damping="0.1" friction="0.1"/> -->
     <limit
       lower="-3.14"
@@ -1548,5 +1489,5 @@
       </material>
     </visual>
-    <collision>
+    <!-- <collision>
       <origin
         xyz="0 0 0"
@@ -1556,5 +1497,5 @@
           filename="package://xingtian/meshes/meshes_s/zqt_yao.STL" />
       </geometry>
-    </collision>
+    </collision> -->
   </link>
   <joint
@@ -1570,13 +1511,4 @@
     <axis
       xyz="0 1 0" />
-    <!-- <sensor name="joint_sensor" type="force_torque">
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